Commit message: update phobos_nuclear urdf

File: urdf/phobos_nuclear.urdf.xacro (robot description, xacro)
@@ -9,6 +9,6 @@
         <xacro:property name="length" value="0.13"/>
         <xacro:property name="mesh_file" value="package://i3dr_phobos_nuclear/mesh/phobos_nuclear.stl"/>
-        <xacro:property name="mesh_offset_xyz" value="0 ${-width/2} 0"/>
-        <xacro:property name="mesh_offset_rpy" value="0 ${pi} ${pi}"/>
+        <xacro:property name="mesh_offset_xyz" value="0 0 0"/>
+        <xacro:property name="mesh_offset_rpy" value="0 0 ${-pi/2}"/>
         <xacro:property name="box_offset_xyz" value="${(length/2)-(height/2)} 0 0"/>
         <xacro:property name="box_offset_rpy" value="0 0 0"/>
@@ -20,10 +20,5 @@
         <link name="${camera_name}_cameraRight" />
         <link name="${camera_name}_depth_optical_frame" />
-        <link name="${camera_name}_base_link" />
-        <link name="${camera_name}_mount_point_1"/>
-        <link name="${camera_name}_mount_point_2"/>
-        <link name="${camera_name}_mount_point_3"/>
-        <link name="${camera_name}_mount_point_4"/>
-        <link name="${camera_name}_center">
+        <link name="${camera_name}_base_link" >
             <visual>
                 <xacro:if value="${(en_mesh == 'true')}">
@@ -48,13 +43,18 @@
             </visual>
         </link>
+        <link name="${camera_name}_mount_point_1"/>
+        <link name="${camera_name}_mount_point_2"/>
+        <link name="${camera_name}_mount_point_3"/>
+        <link name="${camera_name}_mount_point_4"/>
+        <link name="${camera_name}_center"/>
         <joint name="${camera_name}_right_camera_joint" type="fixed">
             <parent link="${camera_name}_center"/>
             <child link="${camera_name}_cameraRight"/>
-            <origin xyz="0 ${-0.125}  0" rpy="0 0 0" />
+            <origin xyz="0 ${-0.125} 0" rpy="0 0 0" />
         </joint>
         <joint name="${camera_name}_left_camera_joint" type="fixed">
             <parent link="${camera_name}_center"/>
             <child link="${camera_name}_cameraLeft"/>
-            <origin xyz="0 ${0.125}  0" rpy="0 0 0" />
+            <origin xyz="0 ${0.125} 0" rpy="0 0 0" />
         </joint>
         <joint name="${camera_name}_left_optical_joint" type="fixed">
@@ -78,25 +78,25 @@
             <parent link="${camera_name}_base_link"/>
             <child link="${camera_name}_center"/>
-            <origin xyz="0 0 ${width/2}" rpy="${pi/2} 0 ${-pi/2}" />
+            <origin xyz="0.017675 0 0.167" rpy="${pi/2} 0 ${-pi/2}" />
         </joint>
         <joint name="${camera_name}_mount_point_1_joint" type="fixed">
             <parent link="${camera_name}_base_link"/>
             <child link="${camera_name}_mount_point_1"/>
-            <origin xyz="0.01547866425452535 0.01547866425452535 0" rpy="0 0 0" />
+            <origin xyz="0.0176775 0.0176775 0" rpy="0 0 0" />
         </joint>
         <joint name="${camera_name}_mount_point_2_joint" type="fixed">
             <parent link="${camera_name}_base_link"/>
             <child link="${camera_name}_mount_point_2"/>
-            <origin xyz="-0.01547866425452535 0.01547866425452535 0" rpy="0 0 0" />
+            <origin xyz="-0.0176775 0.0176775 0" rpy="0 0 0" />
         </joint>
         <joint name="${camera_name}_mount_point_3_joint" type="fixed">
             <parent link="${camera_name}_base_link"/>
             <child link="${camera_name}_mount_point_3"/>
-            <origin xyz="0.01547866425452535 -0.01547866425452535 0" rpy="0 0 0" />
+            <origin xyz="0.0176775 -0.0176775 0" rpy="0 0 0" />
         </joint>
         <joint name="${camera_name}_mount_point_4_joint" type="fixed">
             <parent link="${camera_name}_base_link"/>
             <child link="${camera_name}_mount_point_4"/>
-            <origin xyz="-0.01547866425452535 -0.01547866425452535 0" rpy="0 0 0" />
+            <origin xyz="-0.0176775 -0.0176775 0" rpy="0 0 0" />
         </joint>
     </xacro:macro>

Commit message: Added Gazebo controller

File: urdf/phobos_nuclear.urdf.xacro (robot description, xacro)
@@ -100,4 +100,90 @@
             <origin xyz="-0.0176775 -0.0176775 0" rpy="0 0 0" />
         </joint>
+        <gazebo reference="${camera_name}_cameraLeft">
+            <sensor type="multicamera" name="${camera_name}_camera">
+            <update_rate>0.5</update_rate> <!-- reality 60fps on USB3-->
+            <camera name="left">
+                <horizontal_fov>1.04</horizontal_fov>
+                <image>
+                    <width>752</width>
+                    <height>480</height>
+                    <format>L8</format>
+                </image>
+                <clip>
+                    <near>0.02</near>
+                    <far>300</far>
+                </clip>
+                <noise>
+                    <type>gaussian</type>
+                    <mean>0.0</mean>
+                    <stddev>0.007</stddev>
+                </noise>
+            </camera>
+            <camera name="right">
+                <pose>0 -0.07 0 0 0 0</pose>
+                <horizontal_fov>1.3962634</horizontal_fov>
+                <image>
+                    <width>752</width>
+                    <height>480</height>
+                    <format>L8</format>
+                </image>
+                <clip>
+                    <near>0.02</near>
+                    <far>300</far>
+                </clip>
+                <noise>
+                    <type>gaussian</type>
+                    <mean>0.0</mean>
+                    <stddev>0.007</stddev>
+                </noise>
+            </camera>
+            <plugin name="${camera_name}_camera_controller" filename="libgazebo_ros_multicamera.so">
+                <alwaysOn>true</alwaysOn>
+                <updateRate>0.5</updateRate>
+                <cameraName>${camera_name}</cameraName>
+                <imageTopicName>${camera_name}/image_raw</imageTopicName>
+                <cameraInfoTopicName>${camera_name}/camera_info</cameraInfoTopicName>
+                <frameName>${camera_name}_cameraLeft_optical</frameName>
+                <hackBaseline>0.07</hackBaseline>
+                <distortionK1>0.0</distortionK1>
+                <distortionK2>0.0</distortionK2>
+                <distortionK3>0.0</distortionK3>
+                <distortionT1>0.0</distortionT1>
+                <distortionT2>0.0</distortionT2>
+            </plugin>
+            </sensor>
+        </gazebo>
+        <gazebo reference="${camera_name}_depth_camera">
+            <sensor type="depth" name="${camera_name}_depth_camera">
+            <update_rate>0.5</update_rate>
+            <camera>
+                <horizontal_fov>${62.8 * pi/180.0}</horizontal_fov>
+                <image>
+                <format>R8G8B8</format>
+                <width>640</width>
+                <height>480</height>
+                </image>
+                <clip>
+                <near>0.05</near>
+                <far>12</far>
+                </clip>
+            </camera>
+            <plugin name="${camera_name}_depth_camera_controller" filename="libgazebo_ros_openni_kinect.so">
+                <alwaysOn>true</alwaysOn>
+                <updateRate>0.5</updateRate>
+                <imageTopicName>${camera_name}/image_raw</imageTopicName>
+                <cameraInfoTopicName>${camera_name}/camera_info</cameraInfoTopicName>
+                <depthImageTopicName>${camera_name}/depth/image_raw</depthImageTopicName>
+                <depthImageCameraInfoTopicName>${camera_name}/depth/camera_info</depthImageCameraInfoTopicName>
+                <pointCloudTopicName>${camera_name}/depth/points</pointCloudTopicName>
+                <frameName>${camera_name}_depth_optical_frame</frameName>
+                <distortion_k1>0.0</distortion_k1>
+                <distortion_k2>0.0</distortion_k2>
+                <distortion_k3>0.0</distortion_k3>
+                <distortion_t1>0.0</distortion_t1>
+                <distortion_t2>0.0</distortion_t2>
+            </plugin>
+            </sensor>
+    </gazebo>
     </xacro:macro>
 </robot>

Commit message: Simulation: fixed sim frames and added parameters

File: urdf/phobos_nuclear.urdf.xacro (robot description, xacro)
@@ -15,7 +15,15 @@
         <xacro:property name="toe_in_l" value="0"/>
         <xacro:property name="toe_in_r" value="0"/>
+        <xacro:property name="fov_rad" value="${62.8 * pi/180.0}"/>
+        <xacro:property name="sim_w" value="320"/>
+        <xacro:property name="sim_h" value="240"/>
+        <xacro:property name="sim_rate" value="0.5"/>
+        <xacro:property name="sim3d_w" value="320"/>
+        <xacro:property name="sim3d_h" value="240"/>
+        <xacro:property name="sim3d_rate" value="1"/>
         <link name="${camera_name}_cameraLeft_optical" />
         <link name="${camera_name}_cameraRight_optical" />
         <link name="${camera_name}_cameraLeft" />
+        <link name="${camera_name}_cameraLeft_sim" />
         <link name="${camera_name}_cameraRight" />
         <link name="${camera_name}_depth_optical_frame" />
@@ -64,4 +72,9 @@
             <origin xyz="0 0 0" rpy="${-pi/2} 0 ${(-pi/2)-(toe_in_l * (pi/180))}" />
         </joint>
+        <joint name="${camera_name}_left_sim_joint" type="fixed">
+            <parent link="${camera_name}_cameraLeft"/>
+            <child link="${camera_name}_cameraLeft_sim"/>
+            <origin xyz="0.08 0 0" rpy="0 0 0" />
+        </joint>
         <joint name="${camera_name}_right_optical_joint" type="fixed">
             <parent link="${camera_name}_cameraRight"/>
@@ -71,7 +84,7 @@
         </joint>
         <joint name="${camera_name}_depth_optical_joint" type="fixed">
-            <parent link="${camera_name}_cameraRight"/>
+            <parent link="${camera_name}_cameraLeft_sim"/>
             <child link="${camera_name}_depth_optical_frame"/>
-            <origin xyz="0 0 0" rpy="${-pi/2} 0 ${(-pi/2)}" />
+            <origin xyz="0 0 0" rpy="0 0 0" />
         </joint>
         <joint name="${camera_name}_mount_center_joint" type="fixed">
@@ -100,90 +113,76 @@
             <origin xyz="-0.0176775 -0.0176775 0" rpy="0 0 0" />
         </joint>
-        <gazebo reference="${camera_name}_cameraLeft">
-            <sensor type="multicamera" name="${camera_name}_camera">
-            <update_rate>0.5</update_rate> <!-- reality 60fps on USB3-->
-            <camera name="left">
-                <horizontal_fov>1.04</horizontal_fov>
-                <image>
-                    <width>752</width>
-                    <height>480</height>
-                    <format>L8</format>
-                </image>
-                <clip>
-                    <near>0.02</near>
-                    <far>300</far>
-                </clip>
-                <noise>
-                    <type>gaussian</type>
-                    <mean>0.0</mean>
-                    <stddev>0.007</stddev>
-                </noise>
-            </camera>
-            <camera name="right">
-                <pose>0 -0.07 0 0 0 0</pose>
-                <horizontal_fov>1.3962634</horizontal_fov>
-                <image>
-                    <width>752</width>
-                    <height>480</height>
-                    <format>L8</format>
-                </image>
-                <clip>
-                    <near>0.02</near>
-                    <far>300</far>
-                </clip>
-                <noise>
-                    <type>gaussian</type>
-                    <mean>0.0</mean>
-                    <stddev>0.007</stddev>
-                </noise>
-            </camera>
-            <plugin name="${camera_name}_camera_controller" filename="libgazebo_ros_multicamera.so">
-                <alwaysOn>true</alwaysOn>
-                <updateRate>0.5</updateRate>
-                <cameraName>${camera_name}</cameraName>
-                <imageTopicName>${camera_name}/image_raw</imageTopicName>
-                <cameraInfoTopicName>${camera_name}/camera_info</cameraInfoTopicName>
-                <frameName>${camera_name}_cameraLeft_optical</frameName>
-                <hackBaseline>0.07</hackBaseline>
-                <distortionK1>0.0</distortionK1>
-                <distortionK2>0.0</distortionK2>
-                <distortionK3>0.0</distortionK3>
-                <distortionT1>0.0</distortionT1>
-                <distortionT2>0.0</distortionT2>
-            </plugin>
-            </sensor>
-        </gazebo>
-        <gazebo reference="${camera_name}_depth_camera">
-            <sensor type="depth" name="${camera_name}_depth_camera">
-            <update_rate>0.5</update_rate>
-            <camera>
-                <horizontal_fov>${62.8 * pi/180.0}</horizontal_fov>
-                <image>
-                <format>R8G8B8</format>
-                <width>640</width>
-                <height>480</height>
-                </image>
-                <clip>
-                <near>0.05</near>
-                <far>12</far>
-                </clip>
-            </camera>
-            <plugin name="${camera_name}_depth_camera_controller" filename="libgazebo_ros_openni_kinect.so">
-                <alwaysOn>true</alwaysOn>
-                <updateRate>0.5</updateRate>
-                <imageTopicName>${camera_name}/image_raw</imageTopicName>
-                <cameraInfoTopicName>${camera_name}/camera_info</cameraInfoTopicName>
-                <depthImageTopicName>${camera_name}/depth/image_raw</depthImageTopicName>
-                <depthImageCameraInfoTopicName>${camera_name}/depth/camera_info</depthImageCameraInfoTopicName>
-                <pointCloudTopicName>${camera_name}/depth/points</pointCloudTopicName>
-                <frameName>${camera_name}_depth_optical_frame</frameName>
-                <distortion_k1>0.0</distortion_k1>
-                <distortion_k2>0.0</distortion_k2>
-                <distortion_k3>0.0</distortion_k3>
-                <distortion_t1>0.0</distortion_t1>
-                <distortion_t2>0.0</distortion_t2>
-            </plugin>
-            </sensor>
+    <xacro:macro name="optical_camera" params="name fov_rad:=^ sim_w:=^ sim_h:=^">
+        <camera name="${name}">
+          <horizontal_fov>${fov_rad}</horizontal_fov>
+          <image>
+              <width>${sim_w}</width> <!-- real: 752 -->
+              <height>${sim_h}</height> <!-- real 480 -->
+              <format>L8</format>
+          </image>
+          <clip>
+              <near>0.02</near>
+              <far>300</far>
+          </clip>
+          <noise>
+              <type>gaussian</type>
+              <mean>0.0</mean>
+              <stddev>0.007</stddev>
+          </noise>
+      </camera>
+    </xacro:macro>
+    <gazebo reference="${camera_name}_cameraLeft_sim">
+      <sensor type="multicamera" name="stereo_camera">
+        <update_rate>${sim_rate}</update_rate> <!-- reality 60fps on USB3-->
+        <optical_camera name="left" />
+        <optical_camera name="right" />
+        <plugin name="stereo_camera_controller" filename="libgazebo_ros_multicamera.so">
+          <alwaysOn>true</alwaysOn>
+          <updateRate>${sim_rate}</updateRate>
+          <cameraName>${camera_name}</cameraName>
+          <imageTopicName>image_raw</imageTopicName>
+          <cameraInfoTopicName>camera_info</cameraInfoTopicName>
+          <frameName>${camera_name}_cameraLeft_optical</frameName>
+          <hackBaseline>0.07</hackBaseline>
+          <distortionK1>0.0</distortionK1>
+          <distortionK2>0.0</distortionK2>
+          <distortionK3>0.0</distortionK3>
+          <distortionT1>0.0</distortionT1>
+          <distortionT2>0.0</distortionT2>
+        </plugin>
+      </sensor>
     </gazebo>
-    </xacro:macro>
+    <gazebo reference="${camera_name}_depth_optical_frame">
+      <sensor type="depth" name="${camera_name}_depth_camera">
+        <update_rate>${sim3d_rate}</update_rate>
+        <camera>
+          <horizontal_fov>${fov_rad}</horizontal_fov>
+          <image>
+            <format>R8G8B8</format>
+            <width>${sim3d_w}</width>
+            <height>${sim3d_h}</height>
+          </image>
+          <clip>
+            <near>0.05</near>
+            <far>12</far>
+          </clip>
+        </camera>
+        <plugin name="${camera_name}_depth_camera_controller" filename="libgazebo_ros_openni_kinect.so">
+          <alwaysOn>true</alwaysOn>
+          <updateRate>${sim3d_rate}</updateRate>
+          <imageTopicName>${camera_name}_depth/image_raw</imageTopicName>
+          <cameraInfoTopicName>${camera_name}_depth/camera_info</cameraInfoTopicName>
+          <depthImageTopicName>${camera_name}_depth/depth/image_raw</depthImageTopicName>
+          <depthImageCameraInfoTopicName>${camera_name}_depth/depth/camera_info</depthImageCameraInfoTopicName>
+          <pointCloudTopicName>${camera_name}_depth/depth/points</pointCloudTopicName>
+          <frameName>${camera_name}_cameraLeft_optical</frameName>
+          <distortion_k1>0.0</distortion_k1>
+          <distortion_k2>0.0</distortion_k2>
+          <distortion_k3>0.0</distortion_k3>
+          <distortion_t1>0.0</distortion_t1>
+          <distortion_t2>0.0</distortion_t2>
+        </plugin>
+      </sensor>
+    </gazebo>
+  </xacro:macro>
 </robot>

Commit message: update urdf fixing a few issues

File: urdf/phobos_nuclear.urdf.xacro (robot description, xacro)
@@ -59,10 +59,10 @@
             <parent link="${camera_name}_center"/>
             <child link="${camera_name}_cameraRight"/>
-            <origin xyz="0 ${-0.125} 0" rpy="0 0 0" />
+            <origin xyz="0 ${0.125} 0" rpy="0 0 ${pi/2}" />
         </joint>
         <joint name="${camera_name}_left_camera_joint" type="fixed">
             <parent link="${camera_name}_center"/>
             <child link="${camera_name}_cameraLeft"/>
-            <origin xyz="0 ${0.125} 0" rpy="0 0 0" />
+            <origin xyz="0 ${-0.125} 0" rpy="0 0 ${pi/2}" />
         </joint>
         <joint name="${camera_name}_left_optical_joint" type="fixed">
@@ -91,5 +91,5 @@
             <parent link="${camera_name}_base_link"/>
             <child link="${camera_name}_center"/>
-            <origin xyz="0.017675 0 0.167" rpy="${pi/2} 0 ${-pi/2}" />
+            <origin xyz="0.017675 0 0.167" rpy="${pi/2} 0 0" />
         </joint>
         <joint name="${camera_name}_mount_point_1_joint" type="fixed">

Commit message: updated launcher for new split laser control

File: urdf/phobos_nuclear.urdf.xacro (robot description, xacro)
@@ -44,9 +44,7 @@
                     </xacro:if>
                 </geometry>
-                <xacro:if value="${(en_mesh == 'false')}">
-                    <material name="${camera_name}_camera_colour">
-                        <color rgba="0.1 0.1 0.1 1"/>
-                    </material>
-                </xacro:if>
+                <material name="${camera_name}_camera_colour">
+                    <color rgba="0.1 0.1 0.1 1"/>
+                </material>
             </visual>
         </link>
