Commit message: update camera model

File: urdf/phobos_nuclear.urdf.xacro (robot description, xacro)
@@ -4,15 +4,7 @@
 -->
 <robot xmlns:xacro="http://ros.org/wiki/xacro">
-    <xacro:macro name="i3dr_phobos_nuclear" params="camera_name:=phobos_nuclear en_mesh:=false">
-        <xacro:property name="height" value="0.045"/>
-        <xacro:property name="width" value="0.305"/>
-        <xacro:property name="length" value="0.13"/>
-        <xacro:property name="mesh_file" value="package://i3dr_phobos_nuclear/mesh/phobos_nuclear.stl"/>
-        <xacro:property name="mesh_offset_xyz" value="0 0 0"/>
-        <xacro:property name="mesh_offset_rpy" value="0 0 ${-pi/2}"/>
-        <xacro:property name="box_offset_xyz" value="${(length/2)-(height/2)} 0 0"/>
-        <xacro:property name="box_offset_rpy" value="0 0 0"/>
-        <xacro:property name="toe_in_l" value="0"/>
-        <xacro:property name="toe_in_r" value="0"/>
+    <xacro:macro name="i3dr_phobos_nuclear" params="camera_name:=phobos_nuclear">
+        <xacro:property name="camerabar_mesh_file" value="package://i3dr_phobos_nuclear/mesh/camerabar_s.stl"/>
+        <xacro:property name="interfacing_plate_mesh_file" value="package://i3dr_phobos_nuclear/mesh/interfacing_plate_s.stl"/>
         <xacro:property name="fov_rad" value="${62.8 * pi/180.0}"/>
         <xacro:property name="sim_w" value="320"/>
@@ -28,19 +20,9 @@
         <link name="${camera_name}_cameraRight" />
         <link name="${camera_name}_depth_optical_frame" />
-        <link name="${camera_name}_base_link" >
+        <link name="${camera_name}_interface_plate_link">
             <visual>
-                <xacro:if value="${(en_mesh == 'true')}">
-                    <origin xyz="${mesh_offset_xyz}" rpy="${mesh_offset_rpy}"/>
-                </xacro:if>
-                <xacro:if value="${(en_mesh == 'false')}">
-                    <origin xyz="${box_offset_xyz}" rpy="${box_offset_rpy}"/>
-                </xacro:if>
+                <origin xyz="0 0 0" rpy="0 0 0"/>
                 <geometry>
-                    <xacro:if value="${(en_mesh == 'true')}">
-                        <mesh filename="${mesh_file}"/>
-                    </xacro:if>
-                    <xacro:if value="${(en_mesh == 'false')}">
-                        <box size="${length} ${width} ${height}"/>
-                    </xacro:if>
+                    <mesh filename="${interfacing_plate_mesh_file}"/>
                 </geometry>
                 <material name="${camera_name}_camera_colour">
@@ -49,4 +31,16 @@
             </visual>
         </link>
+        <link name="${camera_name}_camerabar_link">
+            <visual>
+                <origin xyz="0 0 0" rpy="0 0 0"/>
+                <geometry>
+                    <mesh filename="${camerabar_mesh_file}"/>
+                </geometry>
+                <material name="${camera_name}_camera_colour">
+                    <color rgba="0.1 0.1 0.1 1"/>
+                </material>
+            </visual>
+        </link>
+        <link name="${camera_name}_base_link" />
         <link name="${camera_name}_mount_point_1"/>
         <link name="${camera_name}_mount_point_2"/>
@@ -57,10 +51,10 @@
             <parent link="${camera_name}_center"/>
             <child link="${camera_name}_cameraRight"/>
-            <origin xyz="0 ${0.125} 0" rpy="0 0 ${pi/2}" />
+            <origin xyz="${0.125} 0 0" rpy="0 0 0" />
         </joint>
         <joint name="${camera_name}_left_camera_joint" type="fixed">
             <parent link="${camera_name}_center"/>
             <child link="${camera_name}_cameraLeft"/>
-            <origin xyz="0 ${-0.125} 0" rpy="0 0 ${pi/2}" />
+            <origin xyz="${-0.125} 0 0" rpy="0 0 0" />
         </joint>
         <joint name="${camera_name}_left_optical_joint" type="fixed">
@@ -68,5 +62,5 @@
             <child link="${camera_name}_cameraLeft_optical"/>
             <!-- Correct for the optical frame orientation -->
-            <origin xyz="0 0 0" rpy="${-pi/2} 0 ${(-pi/2)-(toe_in_l * (pi/180))}" />
+            <origin xyz="0 0 0" rpy="${-pi/2} 0 0" />
         </joint>
         <joint name="${camera_name}_left_sim_joint" type="fixed">
@@ -79,8 +73,8 @@
             <child link="${camera_name}_cameraRight_optical"/>
             <!-- Correct for the optical frame orientation -->
-            <origin xyz="0 0 0" rpy="${-pi/2} 0 ${(-pi/2)+(toe_in_r * (pi/180))}" />
+            <origin xyz="0 0 0" rpy="${-pi/2} 0 0" />
         </joint>
         <joint name="${camera_name}_depth_optical_joint" type="fixed">
-            <parent link="${camera_name}_cameraLeft_sim"/>
+            <parent link="${camera_name}_cameraLeft_optical"/>
             <child link="${camera_name}_depth_optical_frame"/>
             <origin xyz="0 0 0" rpy="0 0 0" />
@@ -89,5 +83,15 @@
             <parent link="${camera_name}_base_link"/>
             <child link="${camera_name}_center"/>
-            <origin xyz="0.017675 0 0.167" rpy="${pi/2} 0 0" />
+            <origin xyz="0 -0.001 0.175" rpy="${pi/2} ${-pi/2} 0" />
+        </joint>
+        <joint name="${camera_name}_interface_plate_joint" type="fixed">
+            <parent link="${camera_name}_base_link"/>
+            <child link="${camera_name}_interface_plate_link"/>
+            <origin xyz="0 0 0" rpy="0 0 ${pi}" />
+        </joint>
+        <joint name="${camera_name}_camerabar_joint" type="fixed">
+            <parent link="${camera_name}_interface_plate_link"/>
+            <child link="${camera_name}_camerabar_link"/>
+            <origin xyz="0.0223 -0.0186 0.015" rpy="0 0 0" />
         </joint>
         <joint name="${camera_name}_mount_point_1_joint" type="fixed">

File: urdf/phobos_nuclear_scene.urdf.xacro (robot description, xacro)
@@ -9,4 +9,4 @@
     -->
     <xacro:include filename="$(find i3dr_phobos_nuclear)/urdf/phobos_nuclear.urdf.xacro"/>
-    <xacro:i3dr_phobos_nuclear camera_name="phobos_nuclear" en_mesh="true"/>
+    <xacro:i3dr_phobos_nuclear camera_name="phobos_nuclear"/>
 </robot>
