Commit message: add camera name paramters to urdf

File: urdf/phobos_nuclear_scene.urdf.xacro (robot description, xacro)
@@ -5,8 +5,9 @@
 <robot name="phobos_nuclear"
     xmlns:xacro="http://ros.org/wiki/xacro">
-   <!-- <xacro:include filename="$(find i3dr_stereo_camera)/urdf/i3dr_stereo_camera.urdf.xacro" />
-    <xacro:i3dr_stereo_camera camera_name="phobos_nuclear" baseline="0.25" toe_in_r="7" toe_in_l="0" width="0.4" height="0.05" length="0.05" image_width="1920" image_height="1080" image_format="MONO8" hfov="1.04" focus_near="0.3" r="0.1" g="0.1" b="0.1" />
-    -->
-    <xacro:include filename="$(find i3dr_phobos_nuclear)/urdf/phobos_nuclear.urdf.xacro"/>
-    <xacro:i3dr_phobos_nuclear camera_name="phobos_nuclear"/>
+    <xacro:arg name="camera_name" default="phobos_nuclear"/>
+    <!-- <xacro:include filename="$(find i3dr_stereo_camera)/urdf/i3dr_stereo_camera.urdf.xacro" />
+      <xacro:i3dr_stereo_camera camera_name="phobos_nuclear" baseline="0.25" toe_in_r="7" toe_in_l="0" width="0.4" height="0.05" length="0.05" image_width="1920" image_height="1080" image_format="MONO8" hfov="1.04" focus_near="0.3" r="0.1" g="0.1" b="0.1" />
+      -->
+      <xacro:include filename="$(find i3dr_phobos_nuclear)/urdf/phobos_nuclear.urdf.xacro"/>
+      <xacro:i3dr_phobos_nuclear camera_name="$(arg camera_name)"/>
 </robot>
